Commit message: good place to checkpoint dev

File: assets/ros_assets/h1_2_magpie.urdf (robot description, URDF)
Before this commit: robot h1_2_magpie, 50 links, 49 joints
Links:
- link left_wrist_yaw_link: geometry visual mesh filename=../meshes/h1_2/wrist_yaw_link.STL; visual mesh filename=../meshes/magpie/magpie_h12.stl scale=0.001 0.001 0.001
- link right_wrist_yaw_link: geometry visual mesh filename=../meshes/h1_2/wrist_yaw_link.STL; visual mesh filename=../meshes/magpie/magpie_h12.stl scale=0.001 0.001 0.001

File: assets/ros_assets/h1_2_magpie_ros.urdf (robot description, URDF)
Before this commit: robot h1_2_magpie, 53 links, 52 joints
Links:
- link left_wrist_yaw_link: geometry visual mesh filename=package://h12_ros2_model/assets/h1_2/meshes/magpie/magpie_h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 scale=0.001 0.001 0.001; visual mesh filename=package://h12_ros2_model/assets/h1_2/meshes/wrist_yaw_link.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
- link right_wrist_yaw_link: geometry visual mesh filename=package://h12_ros2_model/assets/h1_2/meshes/magpie/magpie_h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 scale=0.001 0.001 0.001; visual mesh filename=package://h12_ros2_model/assets/h1_2/meshes/wrist_yaw_link.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
